Commit message: 调整LW关节力矩限值
将左右髋、大腿和小腿力矩上限设为105Nm，足关节设为25Nm，轮关节设为35Nm。
关节位置与速度限值保持当前文件内容。

File: src/robots/LW_Leg/LW_Leg/urdf/LW.urdf (robot description, URDF)
Before this commit: robot LW, 21 links, 20 joints
Joints:
- joint left_foot_joint: limit lower=-1.919862 upper=1.919862 effort=27.000000 velocity=10.000000 -> lower=-1.919862 upper=1.919862 effort=25.000000 velocity=10.000000
- joint left_hip_joint: limit lower=-1.570796 upper=1.570796 effort=120.000000 velocity=20.000000 -> lower=-1.570796 upper=1.570796 effort=105.000000 velocity=20.000000
- joint left_shank_joint: limit lower=-3.141593 upper=3.141593 effort=120.000000 velocity=20.000000 -> lower=-3.141593 upper=3.141593 effort=105.000000 velocity=20.000000
- joint left_thigh_joint: limit lower=-1.570796 upper=1.570796 effort=120.000000 velocity=20.000000 -> lower=-1.570796 upper=1.570796 effort=105.000000 velocity=20.000000
- joint left_wheel_joint: limit lower=-100.0 upper=100.0 effort=40.000000 velocity=33.000000 -> lower=-100.0 upper=100.0 effort=35.000000 velocity=33.000000
- joint right_foot_joint: limit lower=-1.919862 upper=1.919862 effort=27.000000 velocity=10.000000 -> lower=-1.919862 upper=1.919862 effort=25.000000 velocity=10.000000
- joint right_hip_joint: limit lower=-1.570796 upper=1.570796 effort=120.000000 velocity=20.000000 -> lower=-1.570796 upper=1.570796 effort=105.000000 velocity=20.000000
- joint right_shank_joint: limit lower=-3.141593 upper=3.141593 effort=120.000000 velocity=20.000000 -> lower=-3.141593 upper=3.141593 effort=105.000000 velocity=20.000000
- joint right_thigh_joint: limit lower=-1.570796 upper=1.570796 effort=120.000000 velocity=20.000000 -> lower=-1.570796 upper=1.570796 effort=105.000000 velocity=20.000000
- joint right_wheel_joint: limit lower=-100.0 upper=100.0 effort=40.000000 velocity=33.000000 -> lower=-100.0 upper=100.0 effort=35.000000 velocity=33.000000
